File: hardware/Connectors_Comms.kicad_sch (KiCad schematic)
At the start: 0 parts

Commit message: Schematics Completed
Parts:
- added J2: COMPANION, symbol Connector:Conn_01x03_Pin
- added J3: CAM PWR, symbol Connector:Conn_01x02_Pin
- added J?: SWD Debug, Connector:Tag-Connect_TC2030-IDC-NL_2x03_P1.27mm_Vertical, symbol Connector:Conn_ARM_SWD_TagConnect_TC2030-NL
Connections:
- new net 3V3: J?.1 (VCC)
- new net 5V_CAM: J3.1 (Pin_1)
- new net GND: J2.1 (Pin_1), J3.2 (Pin_2), J?.5 (GND)
- new net RESET: J?.3 (~{RESET})
- new net SWCLK_BOOT0: J?.4 (SWCLK)
- new net SWDIO: J?.2 (SWDIO)
- new net USART2_RX: J2.3 (Pin_3)
- new net USART2_TX: J2.2 (Pin_2)

Commit message: Completed Schematic
Parts:
- gave numbers to parts that had none: 1
- renumbered J2 to J3, J3 to J4
Connections:
- no-connect marks 0 -> 1
Other:
- moved on the sheet: J2, J3, J4

Commit message: Assigned Footprints and Libraries
Parts:
- J3: footprint (none) -> Connector_JST:JST_SH_SM03B-SRSS-TB_1x03-1MP_P1.00mm_Horizontal
- J4: footprint (none) -> Connector_JST:JST_SH_SM02B-SRSS-TB_1x02-1MP_P1.00mm_Horizontal
Changed lines of the file:
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@@
 			)
 		)
-		(property "Footprint" ""
+		(property "Footprint" "Connector_JST:JST_SH_SM03B-SRSS-TB_1x03-1MP_P1.00mm_Horizontal"
 			(at 105.41 130.81 0)
 			(hide yes)
@@
 			)
 		)
-		(property "Footprint" ""
+		(property "Footprint" "Connector_JST:JST_SH_SM02B-SRSS-TB_1x02-1MP_P1.00mm_Horizontal"
 			(at 171.45 125.73 0)
 			(hide yes)
