File: hardware/Current_Sense.kicad_sch (KiCad schematic)
At the start: 0 parts

Commit message: Schematics Completed
Parts:
- added 0.1: R_Shunt1, symbol Device:R_Shunt
- added C13: 0.1uF, symbol Device:C
- added R6, R7: 4.7k, symbol Device:R
- added U4: INA226, Package_SO:TSSOP-10_3x3mm_P0.5mm, symbol Sensor_Energy:INA226
Connections:
- new net 3V3: C13.2, R6.1, R7.1, U4.6 (VS)
- new net 5V: 0.1.4
- new net 5V_CAM: 0.1.1
- new net GND: C13.1, U4.1 (A1), U4.2 (A0), U4.7 (GND)
- new net I2C1_SCL: R7.2, U4.5 (SCL)
- new net I2C1_SDA: R6.2, U4.4 (SDA)
- new net VIN+: 0.1.3, U4.10 (Vin+)
- new net VIN-: 0.1.2, U4.8 (Vbus), U4.9 (Vin-)

Commit message: Completed Schematic
Parts:
- added H1, H2, H3, H4: MountingHole, symbol Mechanical:MountingHole
- added TP1: VBAT, symbol Connector:TestPoint
- added TP2: VBAT_PROT, symbol Connector:TestPoint
- added TP3: 5V, symbol Connector:TestPoint
- added TP4: 3V3, symbol Connector:TestPoint
- added TP5: GND, symbol Connector:TestPoint
- added TP6: RESET, symbol Connector:TestPoint
- renumbered C13 to C17, R6 to R7, R7 to R8
Connections:
- net 3V3: now also TP4.1
- net 5V: now also TP3.1
- net GND: now also TP5.1
- new net RESET: TP6.1
- new net VBAT_PROT: TP2.1
- new net VBAT_RAW: TP1.1
- no-connect marks 0 -> 1
Other:
- moved on the sheet: 0.1, C17, R7, R8, U4

Commit message: Assigned Footprints and Libraries
Parts:
- C17: footprint (none) -> Capacitor_SMD:C_0603_1608Metric
- H1, H2, H3, H4: footprint (none) -> MountingHole:MountingHole_2.2mm_M2
- R7, R8: footprint (none) -> Resistor_SMD:R_0201_0603Metric
- R_Shunt1: renamed from 0.1; value R_Shunt1 -> 0.1; footprint (none) -> Resistor_SMD:R_Shunt_Vishay_WSK2512_6332Metric_T2.21mm
- TP1, TP2, TP3, TP4, TP5, TP6: footprint (none) -> TestPoint:TestPoint_Pad_D1.0mm
Changed lines of the file:
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@@
 			)
 		)
-		(property "Footprint" ""
+		(property "Footprint" "TestPoint:TestPoint_Pad_D1.0mm"
 			(at 228.6 119.38 0)
 			(hide yes)
@@
 			)
 		)
-		(property "Footprint" ""
+		(property "Footprint" "MountingHole:MountingHole_2.2mm_M2"
 			(at 196.85 83.82 0)
 			(hide yes)
@@
 			)
 		)
-		(property "Footprint" ""
+		(property "Footprint" "Resistor_SMD:R_0201_0603Metric"
 			(at 145.542 101.6 90)
 			(hide yes)
@@
 			)
 		)
-		(property "Footprint" ""
+		(property "Footprint" "MountingHole:MountingHole_2.2mm_M2"
 			(at 195.58 69.85 0)
 			(hide yes)
@@
 			)
 		)
-		(property "Footprint" ""
+		(property "Footprint" "TestPoint:TestPoint_Pad_D1.0mm"
 			(at 217.17 119.38 0)
 			(hide yes)
@@
 		(in_pos_files yes)
 		(dnp no)
-		(property "Reference" "0.1"
-			(at 80.01 101.6 0)
+		(property "Reference" "R_Shunt1"
+			(at 83.058 99.568 0)
 			(show_name no)
 			(do_not_autoplace no)
@@
 			)
 		)
-		(property "Value" "R_Shunt1"
-			(at 82.55 99.314 0)
+		(property "Value" "0.1"
+			(at 81.026 101.6 0)
 			(show_name no)
 			(do_not_autoplace no)
@@
 			)
 		)
-		(property "Footprint" ""
+		(property "Footprint" "Resistor_SMD:R_Shunt_Vishay_WSK2512_6332Metric_T2.21mm"
 			(at 83.312 100.33 90)
 			(hide yes)
@@
 			(project "hardware"
 				(path "/cab50fbb-ebde-4823-857c-a8c6585217dd/d4bb029e-f2b4-4211-8168-30cb6e1b2574"
-					(reference "0.1")
+					(reference "R_Shunt1")
 					(unit 1)
 				)
@@
 			)
 		)
-		(property "Footprint" ""
+		(property "Footprint" "MountingHole:MountingHole_2.2mm_M2"
 			(at 217.17 83.82 0)
 			(hide yes)
@@
 			)
 		)
-		(property "Footprint" ""
+		(property "Footprint" "Resistor_SMD:R_0201_0603Metric"
 			(at 153.162 105.41 90)
 			(hide yes)
@@
 			)
 		)
-		(property "Footprint" ""
+		(property "Footprint" "TestPoint:TestPoint_Pad_D1.0mm"
 			(at 220.98 119.38 0)
 			(hide yes)
@@
 			)
 		)
-		(property "Footprint" ""
+		(property "Footprint" "Capacitor_SMD:C_0603_1608Metric"
 			(at 116.84 87.9348 0)
 			(hide yes)
@@
 			)
 		)
-		(property "Footprint" ""
+		(property "Footprint" "TestPoint:TestPoint_Pad_D1.0mm"
 			(at 232.41 119.38 0)
 			(hide yes)
@@
 			)
 		)
-		(property "Footprint" ""
+		(property "Footprint" "TestPoint:TestPoint_Pad_D1.0mm"
 			(at 224.79 119.38 0)
 			(hide yes)
@@
 			)
 		)
-		(property "Footprint" ""
+		(property "Footprint" "TestPoint:TestPoint_Pad_D1.0mm"
 			(at 213.36 119.38 0)
 			(hide yes)
@@
 			)
 		)
-		(property "Footprint" ""
+		(property "Footprint" "MountingHole:MountingHole_2.2mm_M2"
 			(at 215.9 69.85 0)
 			(hide yes)
